File: KiCad/Chimborazo Stratos-1/Chimborazo Stratos-1.kicad_sch (KiCad schematic)
At the start: 21 parts, among them Q1 AO3400A, U1 XIAO-ESP32-C6-SMD

Commit message: reach out
Parts:
- R2: value R -> 100k
Changed lines of the file:
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@@
 			)
 		)
-		(property "Value" "R"
+		(property "Value" "100k"
 			(at 52.07 86.36 90)
 			(show_name no)
